Commit message: primeira vizualização no gazebo

File: src/walle_description/urdf/walle.urdf (robot description, URDF)
Before this commit: robot walle, 4 links, 3 joints
Links:
- removed link caster_wheel
- added link caster, mass 0.01; collision sphere radius=0.02; visual sphere radius=0.02
- link base_link: mass 5.0 -> 1.0
- link left_wheel: mass 0.2 -> 0.1; geometry collision cylinder length=0.05 radius=0.05; visual cylinder length=0.05 radius=0.05
- link right_wheel: mass 0.2 -> 0.1; geometry collision cylinder length=0.05 radius=0.05; visual cylinder length=0.05 radius=0.05
Joints:
- removed joint caster_joint
- removed joint left_wheel_joint
- removed joint right_wheel_joint
- added joint base_to_caster: type fixed, parent base_link, child caster, origin xyz=0 -0.15 -0.05 rpy=0 0 0
- added joint base_to_left_wheel: type continuous, parent base_link, child left_wheel, origin xyz=-0.1 0.25 0 rpy=1.5708 0 0, axis 0 1 0
- added joint base_to_right_wheel: type continuous, parent base_link, child right_wheel, origin xyz=0.1 0.25 0 rpy=1.5708 0 0, axis 0 1 0

Commit message: ajuste de links e roda boba

File: src/walle_description/urdf/walle.urdf (robot description, URDF)
Before this commit: robot walle, 4 links, 3 joints
Links:
- removed link caster
- added link caster_wheel, mass 0.05; collision sphere radius=0.08; visual sphere radius=0.08
- link base_link: mass 1.0 -> 10; geometry collision box size=0.5 0.5 0.15; visual box size=0.75 0.5 0.15
- link left_wheel: geometry collision cylinder length=0.05 radius=0.1; visual cylinder length=0.05 radius=0.1
- link right_wheel: geometry collision cylinder length=0.05 radius=0.1; visual cylinder length=0.05 radius=0.1
Joints:
- removed joint base_to_caster
- removed joint base_to_left_wheel
- removed joint base_to_right_wheel
- added joint caster_joint: type continuous, parent base_link, child caster_wheel, origin xyz=0.25 0 0.03 rpy=0 0 0, axis 0 0 1
- added joint left_wheel_joint: type continuous, parent base_link, child left_wheel, origin xyz=-0.13 0.25 0.05 rpy=0 0 0, axis 0 1 0
- added joint right_wheel_joint: type continuous, parent base_link, child right_wheel, origin xyz=-0.13 -0.25 0.05 rpy=0 0 0, axis 0 1 0

Commit message: primeira movimentação com sensores ultrassonicos

File: src/walle_description/urdf/walle.urdf (robot description, URDF)
Before this commit: robot wallerson, 4 links, 3 joints
Links:
- added link front_ultrasonic_link, mass 0.01; collision cylinder length=0.03 radius=0.02; visual cylinder length=0.03 radius=0.02
- added link rear_ultrasonic_link, mass 0.01; collision cylinder length=0.03 radius=0.02; visual cylinder length=0.03 radius=0.02
- added link sensor_mount, mass 0.1; collision box size=0 0 0; visual box size=0.75 0.2 0.03
- added link webcam_link, mass 0.01; collision box size=0.05 0.03 0.02; visual box size=0.05 0.03 0.02
- link base_link: geometry collision box size=0.75 0.5 0.15; visual box size=0.75 0.5 0.15
Joints:
- added joint front_ultrasonic_joint: type fixed, parent sensor_mount, child front_ultrasonic_link, origin xyz=0.35 0 0.03 rpy=0 0 0
- added joint rear_ultrasonic_joint: type fixed, parent sensor_mount, child rear_ultrasonic_link, origin xyz=-0.35 0 0.03 rpy=0 0 3.14159
- added joint sensor_mount_joint: type fixed, parent base_link, child sensor_mount, origin xyz=0 0 0.23 rpy=0 0 0
- added joint webcam_joint: type fixed, parent sensor_mount, child webcam_link, origin xyz=0.05 0 0.035 rpy=0 0 0
